File: Hardware/Satellite_Transceiver_Function_Board__Swarm_M138.brd (EAGLE design)
At the start: 37.5 x 65 mm, 38 parts, among them J3 MICROMOD_FUNCTION_STANDARD, U1 SWARM_M138_TRANSCEIVER_MAIN, U2 MIC94064/5_MIC94064YC6, U3 EEPROM

Commit message: x01 PCB
Parts:
- added C8: 0.1uF, SparkFun-Capacitors:0603
- added C9: 10uF, SparkFun-Capacitors:0603
- moved C7 1.27 mm to (6.99, 20.3)
- moved R3 1.27 mm to (5.08, 20.3)
Connections:
- net GND: now also C8.2, C9.2
- net VIN: now also C8.1, C9.1
Routing:
- net VIN: track 46.8 -> 52.6 mm
- net GND: track 63.6 -> 66.0 mm, vias 90 -> 91
- net EWP: track 30.6 -> 31.6 mm
- net 3.3V: track 71.7 -> 70.8 mm

Commit message: x03_PCB
Parts:
- C4, C5: device SparkFun-Capacitors:1206-POLAR -> New_Parts:EIA3528
- moved R2 27.4 mm to (8.89, 27.9), flipped to the bottom, turned to 90 degrees
- moved R1 27.3 mm to (8.89, 24.4), flipped to the bottom
- moved GPIO1 26.8 mm to (12.7, 27.6)
- moved U$19 25.6 mm to (12.7, 30.0)
- moved C4 12.2 mm to (-14.7, 15.9), flipped to the bottom, turned to 180 degrees
- moved U$8 8.15 mm to (5.08, 30.0)
- moved C6 7.77 mm to (-15.5, 12.7), flipped to the bottom, turned to 0 degrees
- moved EWP 6.35 mm to (5.08, 28.2)
- moved U3 5.08 mm to (0.00, 25.4)
- moved C7 4.06 mm to (6.99, 24.4), flipped to the bottom
- moved R3 4.06 mm to (5.08, 24.4), flipped to the bottom
- moved U2 2.74 mm to (-10.0, 23.5), flipped to the bottom
- moved C3 2.54 mm to (-14.0, 25.4), flipped to the bottom, turned to 0 degrees
- moved C5 1.82 mm to (-14.7, 19.9), flipped to the bottom, turned to 180 degrees
- moved C1 0.63 mm to (-10.2, 20.7), flipped to the bottom, turned to 180 degrees
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Connections:
- net GND: now also C4.C, C5.C; no longer C4.2, C5.2
- net VCC: now also C4.A, C5.A; no longer C4.1, C5.1
Routing:
- net 3.3V: track 70.8 -> 38.8 mm, vias 4 -> 1
- net GPIO1: track 69.6 -> 41.3 mm, vias 2 -> 3
- net VCC: track 45.7 -> 34.5 mm, vias 2 -> 0
- net GND: track 66.0 -> 55.8 mm, vias 91 -> 95
- net PWR_EN: track 36.6 -> 26.8 mm, vias 2 -> 1
- net SDA: track 24.8 -> 31.0 mm
- net SCL: track 22.4 -> 28.4 mm
- net A2: track 21.7 -> 27.6 mm
- net A1: track 19.9 -> 25.6 mm
- net A0: track 18.8 -> 24.0 mm
- net EWP: track 31.6 -> 36.3 mm, vias 3 -> 2
- net N$14: track 3.84 -> 5.00 mm, vias 1 -> 0
- net VIN: track 52.6 -> 52.5 mm, vias 0 -> 4
- net N$16: track 3.84 -> 3.89 mm, vias 1 -> 0
Other:
- board text added: "x03"
- board text removed: "x01"

Commit message: Delete New_Parts.lbr. Parts are now in the main Eagle libraries
Parts:
- C4, C5: device New_Parts:EIA3528 -> SparkFun-Capacitors:EIA3528
- U2: device New_Parts:SC-70-6 -> SparkFun-IC-Power:SC-70-6
Changed lines of the file:
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@@
 <drawing>
 <settings>
-<setting alwaysvectorfont="yes"/>
+<setting alwaysvectorfont="no"/>
 <setting verticaltext="up"/>
 </settings>
 <grid distance="0.05" unitdist="inch" unit="inch" style="lines" multiple="1" display="yes" altdistance="0.005" altunitdist="inch" altunit="inch"/>
 <layers>
-<layer number="1" name="Top" color="4" fill="1" visible="no" active="yes"/>
-<layer number="16" name="Bottom" color="1" fill="1" visible="no" active="yes"/>
+<layer number="1" name="Top" color="4" fill="1" visible="yes" active="yes"/>
+<layer number="16" name="Bottom" color="1" fill="1" visible="yes" active="yes"/>
 <layer number="17" name="Pads" color="2" fill="1" visible="yes" active="yes"/>
-<layer number="18" name="Vias" color="2" fill="1" visible="no" active="yes"/>
-<layer number="19" name="Unrouted" color="6" fill="1" visible="no" active="yes"/>
+<layer number="18" name="Vias" color="2" fill="1" visible="yes" active="yes"/>
+<layer number="19" name="Unrouted" color="6" fill="1" visible="yes" active="yes"/>
 <layer number="20" name="Dimension" color="24" fill="1" visible="yes" active="yes"/>
 <layer number="21" name="tPlace" color="16" fill="1" visible="yes" active="yes"/>
-<layer number="22" name="bPlace" color="14" fill="1" visible="no" active="yes"/>
-<layer number="23" name="tOrigins" color="15" fill="1" visible="no" active="yes"/>
-<layer number="24" name="bOrigins" color="15" fill="1" visible="no" active="yes"/>
+<layer number="22" name="bPlace" color="14" fill="1" visible="yes" active="yes"/>
+<layer number="23" name="tOrigins" color="15" fill="1" visible="yes" active="yes"/>
+<layer number="24" name="bOrigins" color="15" fill="1" visible="yes" active="yes"/>
 <layer number="25" name="tNames" color="7" fill="1" visible="no" active="yes"/>
 <layer number="26" name="bNames" color="7" fill="1" visible="no" active="yes"/>
@@
 <layer number="43" name="vRestrict" color="2" fill="10" visible="no" active="yes"/>
 <layer number="44" name="Drills" color="7" fill="1" visible="no" active="yes"/>
-<layer number="45" name="Holes" color="7" fill="1" visible="no" active="yes"/>
+<layer number="45" name="Holes" color="7" fill="1" visible="yes" active="yes"/>
 <layer number="46" name="Milling" color="3" fill="1" visible="no" active="yes"/>
-<layer number="47" name="Measures" color="7" fill="1" visible="yes" active="yes"/>
+<layer number="47" name="Measures" color="7" fill="1" visible="no" active="yes"/>
 <layer number="48" name="Document" color="7" fill="1" visible="no" active="yes"/>
 <layer number="49" name="Reference" color="7" fill="1" visible="no" active="yes"/>
@@
 <attribute name="PROD_ID" value="HW-16629" x="12.100559375" y="60.07918125" size="1.778" layer="27" font="vector" ratio="15" display="off"/>
 </element>
-<element name="C4" library="New_Parts" package="EIA3528" value="100uF" x="-14.732" y="15.875" smashed="yes" rot="MR180">
-<attribute name="MANU_PART" value="TPSB107M010R0400" x="-14.732" y="15.875" size="1.778" layer="28" rot="MR180" display="off"/>
+<element name="C4" library="SparkFun-Capacitors" package="EIA3528" value="100uF" x="-14.732" y="15.875" smashed="yes" rot="MR180">
 <attribute name="NAME" x="-14.732" y="14.097" size="0.6096" layer="26" font="vector" ratio="20" rot="MR180" align="bottom-center"/>
-<attribute name="PROD_ID" value="" x="-14.732" y="15.875" size="1.778" layer="28" ratio="15" rot="MR180" display="off"/>
+<attribute name="PROD_ID" value="CAP-16823" x="-14.732" y="15.875" size="1.778" layer="28" ratio="15" rot="MR180" display="off"/>
 <attribute name="VALUE" value="100uF" x="-14.732" y="17.653" size="0.6096" layer="28" font="vector" ratio="20" rot="MR180" align="top-center"/>
 </element>
-<element name="C5" library="New_Parts" package="EIA3528" value="100uF" x="-14.732" y="19.939" smashed="yes" rot="MR180">
-<attribute name="MANU_PART" value="TPSB107M010R0400" x="-14.732" y="19.939" size="1.778" layer="28" rot="MR180" display="off"/>
+<element name="C5" library="SparkFun-Capacitors" package="EIA3528" value="100uF" x="-14.732" y="19.939" smashed="yes" rot="MR180">
 <attribute name="NAME" x="-14.732" y="18.161" size="0.6096" layer="26" font="vector" ratio="20" rot="MR180" align="bottom-center"/>
-<attribute name="PROD_ID" value="" x="-14.732" y="19.939" size="1.778" layer="28" ratio="15" rot="MR180" display="off"/>
+<attribute name="PROD_ID" value="CAP-16823" x="-14.732" y="19.939" size="1.778" layer="28" ratio="15" rot="MR180" display="off"/>
 <attribute name="VALUE" value="100uF" x="-14.732" y="21.717" size="0.6096" layer="28" font="vector" ratio="20" rot="MR180" align="top-center"/>
 </element>
@@
 <attribute name="VALUE" x="-10.16" y="21.463" size="0.6096" layer="28" font="vector" ratio="20" rot="MR180" align="top-center"/>
 </element>
-<element name="U2" library="New_Parts" package="SC-70-6" value="MIC94064/5_MIC94064YC6" x="-10.033" y="23.495" smashed="yes" rot="MR90">
+<element name="U2" library="SparkFun-IC-Power" package="SC-70-6" value="MIC94064/5_MIC94064YC6" x="-10.033" y="23.495" smashed="yes" rot="MR90">
 <attribute name="NAME" x="-8.382" y="22.225" size="1.016" layer="26" rot="MR90"/>
 <attribute name="PROD_ID" value="IC-16794" x="-10.033" y="23.495" size="1.778" layer="28" ratio="15" rot="MR90" display="off"/>

Commit message: x04 PCB
Parts:
- removed LOGO3: OSHW-LOGOM, SparkFun-Aesthetics:OSHW-LOGO-M
- added EN: JUMPER-SMT_2_NO_SILK, SparkFun-Jumpers:SMT-JUMPER_2_NO_SILK
- added R4: 100k, SparkFun-Resistors:0603
- added U$10, U$9: (no value), SparkFun-MicroMod:MICROMOD_LOGO_.5
- added U$11: (no value), output:#EN#0
- LOGO2: value OSHW-LOGOM -> OSHW-LOGOS; device SparkFun-Aesthetics:OSHW-LOGO-M -> SparkFun-Aesthetics:OSHW-LOGO-S
- U2: value MIC94064/5_MIC94064YC6 -> MIC94064YC6
- moved LOGO2 18.0 mm to (12.7, 47.0), flipped to the bottom, turned to 270 degrees
- moved U$1 11.7 mm to (-8.89, 47.0), turned to 270 degrees
- moved U$31 9.92 mm to (7.62, 47.0), turned to 270 degrees
- moved U$2 9.16 mm to (-5.08, 47.0), turned to 90 degrees
- moved U$6 7.41 mm to (6.35, 47.0), turned to 270 degrees
- moved U$40 5.75 mm to (5.71, 47.0), turned to 90 degrees
- moved U$4 4.84 mm to (1.91, 47.0), turned to 90 degrees
- moved U$5 4.84 mm to (-1.91, 47.0), turned to 270 degrees
- moved U$3 4.58 mm to (3.81, 47.0), turned to 90 degrees
- moved U$7 2.54 mm to (0.00, 47.0), turned to 270 degrees
- moved U$41 2.01 mm to (1.91, 47.0), turned to 270 degrees
- moved U$19 1.02 mm to (12.7, 29.0), turned to 270 degrees
- moved U$8 1.02 mm to (5.08, 29.0), turned to 270 degrees
Connections:
- new net N$1: EN.1, R4.1
- net 3.3V: now also EN.2
- net GND: now also J3.2, J3.8
- net PWR_EN: now also R4.2
Routing:
- net 3.3V: track 38.8 -> 64.0 mm
- net PWR_EN: track 26.8 -> 33.3 mm, vias 1 -> 3
- net GND: track 55.8 -> 60.7 mm, vias 95 -> 94
- net N$1: track 0.00 -> 3.23 mm
Other:
- board text added: "x04"
- board text removed: "x03"
