File: Hardware/Satellite_Transceiver_Function_Board__Swarm_M138.sch (EAGLE design)
At the start: 28 parts, among them J3 MICROMOD_FUNCTION_STANDARD, U1 SWARM_M138_TRANSCEIVER_MAIN, U2 MIC94064/5_MIC94064YC6, U3 EEPROM

Commit message: x01 PCB
Parts:
- added C8: 0.1uF, SparkFun-Capacitors:0.1UF-0603-25V-5%
- added C9: 10uF, SparkFun-Capacitors:10UF-0603-6.3V-20%
Connections:
- net GND: now also C8.2, C9.2
- net VIN: now also C8.1, C9.1
Other:
- moved on the sheet: C1, C2
Changed lines of the file:
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@@
 <part name="U2" library="New_Parts" deviceset="MIC94064/5" device="_MIC94064YC6"/>
 <part name="GND5" library="SparkFun-PowerSymbols" deviceset="GND" device=""/>
+<part name="C8" library="SparkFun-Capacitors" deviceset="0.1UF" device="-0603-25V-5%" value="0.1uF"/>
+<part name="GND6" library="SparkFun-PowerSymbols" deviceset="GND" device=""/>
+<part name="GND7" library="SparkFun-PowerSymbols" deviceset="GND" device=""/>
+<part name="SUPPLY8" library="SparkFun-PowerSymbols" deviceset="VIN" device=""/>
+<part name="C9" library="SparkFun-Capacitors" deviceset="10UF" device="-0603-6.3V-20%" value="10uF"/>
+<part name="SUPPLY11" library="SparkFun-PowerSymbols" deviceset="VIN" device=""/>
 </parts>
 <sheets>
@@
 <instance part="FD3" gate="G$1" x="238.76" y="43.18" smashed="yes"/>
 <instance part="FD4" gate="G$1" x="238.76" y="45.72" smashed="yes"/>
-<instance part="C2" gate="G$1" x="48.26" y="50.8" smashed="yes">
-<attribute name="NAME" x="49.784" y="53.721" size="1.778" layer="95" font="vector"/>
-<attribute name="VALUE" x="49.784" y="48.641" size="1.778" layer="96" font="vector"/>
-</instance>
-<instance part="GND19" gate="1" x="27.94" y="43.18" smashed="yes">
-<attribute name="VALUE" x="27.94" y="42.926" size="1.778" layer="96" font="vector" align="top-center"/>
-</instance>
-<instance part="GND20" gate="1" x="48.26" y="43.18" smashed="yes">
-<attribute name="VALUE" x="48.26" y="42.926" size="1.778" layer="96" font="vector" align="top-center"/>
+<instance part="C2" gate="G$1" x="22.86" y="50.8" smashed="yes">
+<attribute name="NAME" x="24.384" y="53.721" size="1.778" layer="95" font="vector"/>
+<attribute name="VALUE" x="24.384" y="48.641" size="1.778" layer="96" font="vector"/>
+</instance>
+<instance part="GND19" gate="1" x="33.02" y="43.18" smashed="yes">
+<attribute name="VALUE" x="33.02" y="42.926" size="1.778" layer="96" font="vector" align="top-center"/>
+</instance>
+<instance part="GND20" gate="1" x="22.86" y="43.18" smashed="yes">
+<attribute name="VALUE" x="22.86" y="42.926" size="1.778" layer="96" font="vector" align="top-center"/>
 </instance>
 <instance part="C3" gate="G$1" x="22.86" y="22.86" smashed="yes">
@@
 <instance part="U$1" gate="G$1" x="172.72" y="45.72" smashed="yes"/>
 <instance part="U$2" gate="G$1" x="172.72" y="45.72" smashed="yes"/>
-<instance part="SUPPLY16" gate="G$1" x="48.26" y="58.42" smashed="yes">
-<attribute name="VALUE" x="48.26" y="61.214" size="1.778" layer="96" align="bottom-center"/>
+<instance part="SUPPLY16" gate="G$1" x="22.86" y="58.42" smashed="yes">
+<attribute name="VALUE" x="22.86" y="61.214" size="1.778" layer="96" align="bottom-center"/>
 </instance>
 <instance part="H5" gate="G1" x="167.64" y="157.48" smashed="yes">
@@
 <attribute name="REV" x="236.22" y="6.604" size="2.7432" layer="94" font="vector"/>
 </instance>
-<instance part="C1" gate="G$1" x="27.94" y="50.8" smashed="yes">
-<attribute name="NAME" x="29.464" y="53.721" size="1.778" layer="95" font="vector"/>
-<attribute name="VALUE" x="29.464" y="48.641" size="1.778" layer="96" font="vector"/>
-</instance>
-<instance part="SUPPLY7" gate="G$1" x="27.94" y="58.42" smashed="yes">
-<attribute name="VALUE" x="27.94" y="61.214" size="1.778" layer="96" align="bottom-center"/>
+<instance part="C1" gate="G$1" x="33.02" y="50.8" smashed="yes">
+<attribute name="NAME" x="34.544" y="53.721" size="1.778" layer="95" font="vector"/>
+<attribute name="VALUE" x="34.544" y="48.641" size="1.778" layer="96" font="vector"/>
+</instance>
+<instance part="SUPPLY7" gate="G$1" x="33.02" y="58.42" smashed="yes">
+<attribute name="VALUE" x="33.02" y="61.214" size="1.778" layer="96" align="bottom-center"/>
 </instance>
 <instance part="U2" gate="U1" x="114.3" y="48.26" smashed="yes">
@@
 <instance part="GND5" gate="1" x="101.6" y="38.1" smashed="yes">
 <attribute name="VALUE" x="101.6" y="37.846" size="1.778" layer="96" font="vector" align="top-center"/>
+</instance>
+<instance part="C8" gate="G$1" x="53.34" y="50.8" smashed="yes">
+<attribute name="NAME" x="54.864" y="53.721" size="1.778" layer="95" font="vector"/>
+<attribute name="VALUE" x="54.864" y="48.641" size="1.778" layer="96" font="vector"/>
+</instance>
+<instance part="GND6" gate="1" x="43.18" y="43.18" smashed="yes">
+<attribute name="VALUE" x="43.18" y="42.926" size="1.778" layer="96" font="vector" align="top-center"/>
+</instance>
+<instance part="GND7" gate="1" x="53.34" y="43.18" smashed="yes">
+<attribute name="VALUE" x="53.34" y="42.926" size="1.778" layer="96" font="vector" align="top-center"/>
+</instance>
+<instance part="SUPPLY8" gate="G$1" x="53.34" y="58.42" smashed="yes">
+<attribute name="VALUE" x="53.34" y="61.214" size="1.778" layer="96" align="bottom-center"/>
+</instance>
+<instance part="C9" gate="G$1" x="43.18" y="50.8" smashed="yes">
+<attribute name="NAME" x="44.704" y="53.721" size="1.778" layer="95" font="vector"/>
+<attribute name="VALUE" x="44.704" y="48.641" size="1.778" layer="96" font="vector"/>
+</instance>
+<instance part="SUPPLY11" gate="G$1" x="43.18" y="58.42" smashed="yes">
+<attribute name="VALUE" x="43.18" y="61.214" size="1.778" layer="96" align="bottom-center"/>
 </instance>
 </instances>
@@
 <pinref part="GND19" gate="1" pin="GND"/>
 <pinref part="C1" gate="G$1" pin="2"/>
-<wire x1="27.94" y1="45.72" x2="27.94" y2="48.26" width="0.1524" layer="91"/>
+<wire x1="33.02" y1="45.72" x2="33.02" y2="48.26" width="0.1524" layer="91"/>
 </segment>
 <segment>
 <pinref part="GND20" gate="1" pin="GND"/>
 <pinref part="C2" gate="G$1" pin="2"/>
-<wire x1="48.26" y1="45.72" x2="48.26" y2="48.26" width="0.1524" layer="91"/>
+<wire x1="22.86" y1="45.72" x2="22.86" y2="48.26" width="0.1524" layer="91"/>
 </segment>
 <segment>
@@
 <wire x1="101.6" y1="43.18" x2="101.6" y2="40.64" width="0.1524" layer="91"/>
 </segment>
+<segment>
+<pinref part="GND6" gate="1" pin="GND"/>
+<pinref part="C9" gate="G$1" pin="2"/>
+<wire x1="43.18" y1="45.72" x2="43.18" y2="48.26" width="0.1524" layer="91"/>
+</segment>
+<segment>
+<pinref part="GND7" gate="1" pin="GND"/>
+<pinref part="C8" gate="G$1" pin="2"/>
+<wire x1="53.34" y1="45.72" x2="53.34" y2="48.26" width="0.1524" layer="91"/>
+</segment>
 </net>
 <net name="VCC" class="0">
@@
 <pinref part="C2" gate="G$1" pin="1"/>
 <pinref part="SUPPLY16" gate="G$1" pin="VIN"/>
-<wire x1="48.26" y1="55.88" x2="48.26" y2="58.42" width="0.1524" layer="91"/>
+<wire x1="22.86" y1="55.88" x2="22.86" y2="58.42" width="0.1524" layer="91"/>
 </segment>
 <segment>
@@
 <pinref part="C1" gate="G$1" pin="1"/>
 <pinref part="SUPPLY7" gate="G$1" pin="VIN"/>
-<wire x1="27.94" y1="55.88" x2="27.94" y2="58.42" width="0.1524" layer="91"/>
+<wire x1="33.02" y1="55.88" x2="33.02" y2="58.42" width="0.1524" layer="91"/>
 </segment>
 <segment>
@@
 <wire x1="127" y1="53.34" x2="127" y2="55.88" width="0.1524" layer="91"/>
 </segment>
-</net>
+<segment>
+<pinref part="C8" gate="G$1" pin="1"/>
+<pinref part="SUPPLY8" gate="G$1" pin="VIN"/>
+<wire x1="53.34" y1="55.88" x2="53.34" y2="58.42" width="0.1524" layer="91"/>
+</segment>
+<segment>
+<pinref part="C9" gate="G$1" pin="1"/>
+<pinref part="SUPPLY11" gate="G$1" pin="VIN"/>
+<wire x1="43.18" y1="55.88" x2="43.18" y2="58.42" width="0.1524" layer="91"/>
+</segment>
+</net>

Commit message: x03_PCB
Parts:
- C4, C5: device SparkFun-Capacitors:100UF-POLAR-1206-6.3V-20%(TANT) -> New_Parts:100UF-POLAR-EIA3528-10V-20%
Other:
- note added: "VIN: Min: 1.7V Max: 5.5V"
- note added: "VIN: Min: 3.0V Max: 5.0V"
- note added: "x03"
- note removed: "VIN: Min: 3.00V Max: 5.00V"
- note removed: "x01"
Changed lines of the file:
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@@
 <part name="GND24" library="SparkFun-PowerSymbols" deviceset="GND" device=""/>
 <part name="GND25" library="SparkFun-PowerSymbols" deviceset="GND" device=""/>
-<part name="C4" library="SparkFun-Capacitors" deviceset="100UF-POLAR" device="-1206-6.3V-20%(TANT)" value="100uF"/>
-<part name="C5" library="SparkFun-Capacitors" deviceset="100UF-POLAR" device="-1206-6.3V-20%(TANT)" value="100uF"/>
+<part name="C4" library="New_Parts" deviceset="100UF-POLAR" device="-EIA3528-10V-20%" value="100uF"/>
+<part name="C5" library="New_Parts" deviceset="100UF-POLAR" device="-EIA3528-10V-20%" value="100uF"/>
 <part name="U1" library="SparkFun-RF" deviceset="SWARM_M138_TRANSCEIVER" device="_MAIN"/>
 <part name="SUPPLY19" library="SparkFun-PowerSymbols" deviceset="3.3V" device=""/>
@@
 <sheet>
 <plain>
-<text x="240.03" y="6.35" size="2.54" layer="94" font="vector">x01</text>
+<text x="240.03" y="6.35" size="2.54" layer="94" font="vector">x03</text>
 <text x="168.91" y="8.89" size="2.54" layer="94" font="vector">Paul Clark</text>
 <text x="83.82" y="81.28" size="2.54" layer="94" font="vector">Power Switch</text>
@@
 <wire x1="132.08" y1="185.42" x2="132.08" y2="88.9" width="0.1524" layer="97" style="longdash"/>
 <text x="137.16" y="177.8" size="2.54" layer="94" font="vector">Swarm M138</text>
-<text x="139.7" y="142.24" size="2.032" layer="97" font="vector" align="top-left">VIN:
-Min: 3.00V
-Max: 5.00V
+<text x="142.24" y="142.24" size="2.032" layer="97" font="vector" align="top-left">VIN:
+Min: 3.0V
+Max: 5.0V
 </text>
-<text x="139.7" y="106.68" size="2.032" layer="97" font="vector" align="top-left">Current Draw @ 3.3V:
+<text x="142.24" y="106.68" size="2.032" layer="97" font="vector" align="top-left">Current Draw @ 3.3V:
 Sleep: Modem: 80µA Peak
 RX: 26mA Typ. / 40mA Peak
 TX: 850mA Typ. / 1000mA Peak
 </text>
-<text x="190.5" y="106.68" size="2.032" layer="97" font="vector" align="top-left">Current Draw @ 5.0V:
+<text x="193.04" y="106.68" size="2.032" layer="97" font="vector" align="top-left">Current Draw @ 5.0V:
 Sleep: Modem: 110µA Peak
 RX: 25mA Typ. / 45mA Peak
@@
 <wire x1="78.74" y1="88.9" x2="78.74" y2="0" width="0.1524" layer="97" style="longdash"/>
 <wire x1="147.32" y1="88.9" x2="147.32" y2="35.56" width="0.1524" layer="97" style="longdash"/>
+<text x="106.68" y="33.02" size="2.032" layer="97" font="vector" align="top-left">VIN:
+Min: 1.7V
+Max: 5.5V
+</text>
 </plain>
 <instances>

Commit message: Delete New_Parts.lbr. Parts are now in the main Eagle libraries
Parts:
- C4, C5: device New_Parts:100UF-POLAR-EIA3528-10V-20% -> SparkFun-Capacitors:100UF-POLAR-EIA3528-10V-20%(TANT)
- U2: device New_Parts:MIC94064/5_MIC94064YC6 -> SparkFun-IC-Power:MIC94064/5_MIC94064YC6
Changed lines of the file:
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@@
 <part name="GND24" library="SparkFun-PowerSymbols" deviceset="GND" device=""/>
 <part name="GND25" library="SparkFun-PowerSymbols" deviceset="GND" device=""/>
-<part name="C4" library="New_Parts" deviceset="100UF-POLAR" device="-EIA3528-10V-20%" value="100uF"/>
-<part name="C5" library="New_Parts" deviceset="100UF-POLAR" device="-EIA3528-10V-20%" value="100uF"/>
+<part name="C4" library="SparkFun-Capacitors" deviceset="100UF-POLAR" device="-EIA3528-10V-20%(TANT)" value="100uF"/>
+<part name="C5" library="SparkFun-Capacitors" deviceset="100UF-POLAR" device="-EIA3528-10V-20%(TANT)" value="100uF"/>
 <part name="U1" library="SparkFun-RF" deviceset="SWARM_M138_TRANSCEIVER" device="_MAIN"/>
 <part name="SUPPLY19" library="SparkFun-PowerSymbols" deviceset="3.3V" device=""/>
@@
 <part name="C1" library="SparkFun-Capacitors" deviceset="10UF" device="-0603-6.3V-20%" value="10uF"/>
 <part name="SUPPLY7" library="SparkFun-PowerSymbols" deviceset="VIN" device=""/>
-<part name="U2" library="New_Parts" deviceset="MIC94064/5" device="_MIC94064YC6"/>
+<part name="U2" library="SparkFun-IC-Power" deviceset="MIC94064/5" device="_MIC94064YC6"/>
 <part name="GND5" library="SparkFun-PowerSymbols" deviceset="GND" device=""/>
 <part name="C8" library="SparkFun-Capacitors" deviceset="0.1UF" device="-0603-25V-5%" value="0.1uF"/>

Commit message: x04 PCB
Parts:
- removed LOGO3: OSHW-LOGOM, SparkFun-Aesthetics:OSHW-LOGOM
- added EN: JUMPER-SMT_2_NO_SILK, SparkFun-Jumpers:JUMPER-SMT_2_NO_SILK
- added R4: 100k, SparkFun-Resistors:100KOHM-0603-1/10W-1%
- LOGO2: value OSHW-LOGOM -> OSHW-LOGOS; device SparkFun-Aesthetics:OSHW-LOGOM -> SparkFun-Aesthetics:OSHW-LOGOS
- U2: value MIC94064/5_MIC94064YC6 -> MIC94064YC6
Connections:
- new net N$1: EN.1, R4.1
- net 3.3V: now also EN.2
- net PWR_EN: now also R4.2
Other:
- note added: "Close jumper to enable modem power (when PWR_EN is not connected)"
- note added: "x04"
- note removed: "x03"
- moved on the sheet: U2
