File: Hardware/Production/Satellite_Transceiver_Function_Board__Swarm_M138-Panel.brd (EAGLE design)
At the start: 133.6 x 149.6 mm, 234 parts, among them J1 MICROMOD_FUNCTION_STANDARD, J2 MICROMOD_FUNCTION_STANDARD, J3 MICROMOD_FUNCTION_STANDARD, J4 MICROMOD_FUNCTION_STANDARD, J5 MICROMOD_FUNCTION_STANDARD, J6 MICROMOD_FUNCTION_STANDARD, U1 SWARM_M138_TRANSCEIVER_MAIN, U10 SWARM_M138_TRANSCEIVER_MAIN, U11 EEPROM, U12 MIC94064/5_MIC94064YC6, U13 SWARM_M138_TRANSCEIVER_MAIN, U14 EEPROM, U15 MIC94064/5_MIC94064YC6, U16 SWARM_M138_TRANSCEIVER_MAIN, U17 EEPROM, U18 MIC94064/5_MIC94064YC6, U2 MIC94064/5_MIC94064YC6, U3 EEPROM, U4 SWARM_M138_TRANSCEIVER_MAIN, U5 EEPROM, U6 MIC94064/5_MIC94064YC6, U7 SWARM_M138_TRANSCEIVER_MAIN, U8 EEPROM, U9 MIC94064/5_MIC94064YC6

Commit message: x03_PCB
Parts:
- C13, C14, C22, C23, C31, C32, C4, C40, C41, C49, C5, C50: device SparkFun-Capacitors:1206-POLAR -> New_Parts:EIA3528
- moved R17 27.4 mm to (85.9, 108.4), flipped to the bottom, turned to 270 degrees
- moved R8 27.4 mm to (103.6, 27.9), flipped to the bottom, turned to 90 degrees
- moved R2 27.4 mm to (27.6, 27.9), flipped to the bottom, turned to 90 degrees
- moved R5 27.4 mm to (65.6, 27.9), flipped to the bottom, turned to 90 degrees
- moved R11 27.4 mm to (9.86, 108.4), flipped to the bottom, turned to 270 degrees
- moved R14 27.4 mm to (47.9, 108.4), flipped to the bottom, turned to 270 degrees
- moved R16 27.3 mm to (85.9, 112.0), flipped to the bottom
- moved R7 27.3 mm to (103.6, 24.4), flipped to the bottom
- moved R1 27.3 mm to (27.6, 24.4), flipped to the bottom
- moved R10 27.3 mm to (9.86, 112.0), flipped to the bottom
- moved R13 27.3 mm to (47.9, 112.0), flipped to the bottom
- moved R4 27.3 mm to (65.6, 24.4), flipped to the bottom
- moved GPIO3 26.8 mm to (107.4, 27.6)
- moved GPIO4 26.8 mm to (6.05, 108.8)
- moved GPIO1 26.8 mm to (31.4, 27.6)
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Connections:
- net GND: now also C4.C, C5.C; no longer C4.2, C5.2
- net GND1: now also C13.C, C14.C; no longer C13.2, C14.2
- net GND2: now also C22.C, C23.C; no longer C22.2, C23.2
- net GND3: now also C31.C, C32.C; no longer C31.2, C32.2
- net GND4: now also C40.C, C41.C; no longer C40.2, C41.2
- net GND5: now also C49.C, C50.C; no longer C49.2, C50.2
- net VCC: now also C4.A, C5.A; no longer C4.1, C5.1
- net VCC1: now also C13.A, C14.A; no longer C13.1, C14.1
- net VCC2: now also C22.A, C23.A; no longer C22.1, C23.1
- net VCC3: now also C31.A, C32.A; no longer C31.1, C32.1
- net VCC4: now also C40.A, C41.A; no longer C40.1, C41.1
- net VCC5: now also C49.A, C50.A; no longer C49.1, C50.1
Routing:
- net 3.3V5: track 70.8 -> 38.8 mm, vias 4 -> 1
- net 3.3V1: track 70.8 -> 38.8 mm, vias 4 -> 1
- net 3.3V: track 70.8 -> 38.8 mm, vias 4 -> 1
- net 3.3V4: track 70.8 -> 38.8 mm, vias 4 -> 1
- net 3.3V3: track 70.8 -> 38.8 mm, vias 4 -> 1
- net 3.3V2: track 70.8 -> 38.8 mm, vias 4 -> 1
- net GPIO2: track 69.6 -> 41.3 mm, vias 2 -> 3
- net GPIO1: track 69.6 -> 41.3 mm, vias 2 -> 3
- net GPIO6: track 69.6 -> 41.3 mm, vias 2 -> 3
- net GPIO4: track 69.6 -> 41.3 mm, vias 2 -> 3
- net GPIO3: track 69.6 -> 41.3 mm, vias 2 -> 3
- net GPIO5: track 69.6 -> 41.3 mm, vias 2 -> 3
- net VCC2: track 45.7 -> 34.5 mm, vias 2 -> 0
- net VCC4: track 45.7 -> 34.5 mm, vias 2 -> 0
- net VCC3: track 45.7 -> 34.5 mm, vias 2 -> 0
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Other:
- board text added: "x03"
- board text removed: "x01"

Commit message: Delete New_Parts.lbr. Parts are now in the main Eagle libraries
Parts:
- C13, C14, C22, C23, C31, C32, C4, C40, C41, C49, C5, C50: device New_Parts:EIA3528 -> SparkFun-Capacitors:EIA3528
- U12, U15, U18, U2, U6, U9: device New_Parts:SC-70-6 -> SparkFun-IC-Power:SC-70-6

Commit message: x04 PCB
Parts:
- removed LOGO10, LOGO11, LOGO12, LOGO7, LOGO8, LOGO9: OSHW-LOGOM, SparkFun-Aesthetics:OSHW-LOGO-M
- added EN, EN1, EN2, EN3, EN4, EN5: JUMPER-SMT_2_NO_SILK, SparkFun-Jumpers:SMT-JUMPER_2_NO_SILK
- added R19, R20, R21, R22, R23, R24: 100k, SparkFun-Resistors:0603
- added U$73, U$74, U$88, U$89: (no value), SparkFun-MicroMod:MICROMOD_LOGO_.5
- added U$75, U$90: (no value), output:#EN#0
- added U$76, U$77: SPARKX-LOGO5, SparkX:SPARKX-LARGE
- added U$78: (no value), output:#GPIO1#0
- added U$79, U$80: (no value), output:SWARM_M1381
- added U$81: (no value), output:PLEASE_CONSULT_THE_DOCUMENTATION0
- added U$82: (no value), output:FOR_THE_PEAK_TRANSMIT_CURRENT1
- added U$83, U$86: (no value), output:FUNCTION_BOARD0
- added U$84, U$85: (no value), output:SATELLITE_TRANSCEIVER0
- added U$87: (no value), output:#EWP#0
- LOGO1, LOGO2, LOGO3, LOGO4, LOGO5, LOGO6: value OSHW-LOGOM -> OSHW-LOGOS; device SparkFun-Aesthetics:OSHW-LOGO-M -> SparkFun-Aesthetics:OSHW-LOGO-S
- U$10, U$9: value SPARKX-LOGO5 -> (none); device SparkX:SPARKX-LARGE -> SparkFun-MicroMod:MICROMOD_LOGO_.5
- U$11: device output:#GPIO1#0 -> output:#EN#0
- U$12, U$13: value (none) -> SPARKX-LOGO5; device output:SWARM_M1381 -> SparkX:SPARKX-LARGE
- U$14: device output:PLEASE_CONSULT_THE_DOCUMENTATION0 -> output:#GPIO1#0
- U$15: device output:FOR_THE_PEAK_TRANSMIT_CURRENT1 -> output:SWARM_M1381
- U$16, U$33: device output:FUNCTION_BOARD0 -> output:SWARM_M1381
- U$17: device output:SATELLITE_TRANSCEIVER0 -> output:PLEASE_CONSULT_THE_DOCUMENTATION0
- U$18: device output:SATELLITE_TRANSCEIVER0 -> output:FOR_THE_PEAK_TRANSMIT_CURRENT1
- U$21: device output:#EWP#0 -> output:SATELLITE_TRANSCEIVER0
- U$22: value SPARKX-LOGO5 -> (none); device SparkX:SPARKX-LARGE -> output:SATELLITE_TRANSCEIVER0
- U$23, U$36: value SPARKX-LOGO5 -> (none); device SparkX:SPARKX-LARGE -> output:FUNCTION_BOARD0
- U$24: device output:#GPIO1#0 -> output:#EWP#0
- U$25, U$26: device output:SWARM_M1381 -> SparkFun-MicroMod:MICROMOD_LOGO_.5
- U$27: device output:PLEASE_CONSULT_THE_DOCUMENTATION0 -> output:#EN#0
- U$28: value (none) -> SPARKX-LOGO5; device output:FOR_THE_PEAK_TRANSMIT_CURRENT1 -> SparkX:SPARKX-LARGE
- U$29, U$47: value (none) -> SPARKX-LOGO5; device output:FUNCTION_BOARD0 -> SparkX:SPARKX-LARGE
- U$30: device output:SATELLITE_TRANSCEIVER0 -> output:#GPIO1#0
- U$32: device output:SATELLITE_TRANSCEIVER0 -> output:SWARM_M1381
- U$34: device output:#EWP#0 -> output:PLEASE_CONSULT_THE_DOCUMENTATION0
- U$35: value SPARKX-LOGO5 -> (none); device SparkX:SPARKX-LARGE -> output:FOR_THE_PEAK_TRANSMIT_CURRENT1
- U$37: device output:#GPIO1#0 -> output:SATELLITE_TRANSCEIVER0
- U$38: device output:SWARM_M1381 -> output:SATELLITE_TRANSCEIVER0
- U$39, U$53: device output:SWARM_M1381 -> output:FUNCTION_BOARD0
- U$42: device output:PLEASE_CONSULT_THE_DOCUMENTATION0 -> output:#EWP#0
- U$43: device output:FOR_THE_PEAK_TRANSMIT_CURRENT1 -> SparkFun-MicroMod:MICROMOD_LOGO_.5
- U$44, U$59: device output:FUNCTION_BOARD0 -> SparkFun-MicroMod:MICROMOD_LOGO_.5
- U$45: device output:SATELLITE_TRANSCEIVER0 -> output:#EN#0
- U$46: value (none) -> SPARKX-LOGO5; device output:SATELLITE_TRANSCEIVER0 -> SparkX:SPARKX-LARGE
- U$48: device output:#EWP#0 -> output:#GPIO1#0
- U$49, U$50: value SPARKX-LOGO5 -> (none); device SparkX:SPARKX-LARGE -> output:SWARM_M1381
- U$51: device output:#GPIO1#0 -> output:PLEASE_CONSULT_THE_DOCUMENTATION0
- U$52: device output:SWARM_M1381 -> output:FOR_THE_PEAK_TRANSMIT_CURRENT1
- U$54: device output:PLEASE_CONSULT_THE_DOCUMENTATION0 -> output:SATELLITE_TRANSCEIVER0
- U$55: device output:FOR_THE_PEAK_TRANSMIT_CURRENT1 -> output:SATELLITE_TRANSCEIVER0
- U$57: device output:SATELLITE_TRANSCEIVER0 -> output:#EWP#0
- U$58: device output:SATELLITE_TRANSCEIVER0 -> SparkFun-MicroMod:MICROMOD_LOGO_.5
- U$60: device output:#EWP#0 -> output:#EN#0
- U12, U15, U18, U2, U6, U9: value MIC94064/5_MIC94064YC6 -> MIC94064YC6
- moved R10 125.9 mm to (103.6, 27.9)
- moved R11 123.1 mm to (99.8, 24.4), turned to 90 degrees
- moved U$37 108.3 mm to (96.6, 47.0), flipped to the top, turned to 90 degrees
- moved R12 107.5 mm to (80.8, 27.9), turned to 0 degrees
- moved U$42 103.4 mm to (99.8, 29.0), turned to 270 degrees
- moved U$35 90.6 mm to (102.4, 47.0), turned to 270 degrees
- moved LOGO3 89.6 mm to (107.4, 47.0), turned to 270 degrees
- moved U$43 89.2 mm to (93.5, 47.0), flipped to the top, turned to 90 degrees
- moved U$36 87.0 mm to (98.6, 47.0), turned to 90 degrees
- moved U$39 86.7 mm to (94.7, 47.0), turned to 270 degrees
- moved U$45 86.4 mm to (84.6, 29.0), flipped to the bottom, turned to 270 degrees
- moved U$38 85.0 mm to (92.8, 47.0), flipped to the bottom, turned to 270 degrees
- moved U$44 81.3 mm to (89.7, 47.0), flipped to the bottom, turned to 270 degrees
- moved R4 61.0 mm to (4.78, 27.9), turned to 0 degrees
- moved U$11 60.9 mm to (8.59, 29.0), turned to 270 degrees
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Connections:
- new net N$11: GPIO5.3, R17.1
- new net N$12: GPIO5.1, R18.2
- new net N$13: EN4.1, R20.1
- new net N$15: GPIO6.3, R21.1
- new net N$17: GPIO6.1, R22.2
- new net N$18: EN5.1, R24.1
- net 3.3V: now also EN.2
- net 3.3V1: now also EN1.2, R5.2, R7.1; no longer R4.2, R6.1
- net 3.3V2: now also EN2.2, R11.1, R9.2; no longer R7.2, R9.1
- net 3.3V3: now also EN3.2, R13.2, R15.1; no longer R10.2, R12.1
- net 3.3V4: now also EN4.2, R17.2, R19.1; no longer R13.2, R15.1
- net 3.3V5: now also EN5.2, R21.2, R23.1; no longer R16.2, R18.1
- net EWP1: now also R7.2; no longer R6.2
- net EWP2: now also R11.2; no longer R9.2
- net EWP3: now also R15.2; no longer R12.2
- net EWP4: now also R19.2; no longer R15.2
- net EWP5: now also R23.2; no longer R18.2
- net GND: now also J3.2, J3.8
- net GND1: now also J1.2, J1.8, R6.1; no longer R5.1
- net GND2: now also J2.2, J2.8, R10.1; no longer R8.1
- net GND3: now also J4.2, J4.8, R14.1; no longer R11.1
- net GND4: now also J5.2, J5.8, R18.1; no longer R14.1
- net GND5: now also J6.2, J6.8, R22.1; no longer R17.1
- net N$1: now also EN.1; no longer GPIO2.3
- net N$10: now also EN3.1, R16.1; no longer GPIO6.1, R17.2
- net N$2: now also GPIO2.3, R5.1; no longer GPIO2.1, R5.2
- net N$3: now also GPIO2.1, R6.2; no longer GPIO3.3, R7.1
- net N$4: now also EN1.1, R8.1; no longer GPIO3.1, R8.2
- net N$5: now also GPIO3.3, R9.1; no longer GPIO4.3, R10.1
- net N$6: now also GPIO3.1, R10.2; no longer GPIO4.1, R11.2
- net N$7: now also EN2.1, R12.1; no longer GPIO5.3, R13.1
- net N$8: now also GPIO4.3, R13.1; no longer GPIO5.1, R14.2
- net N$9: now also GPIO4.1, R14.2; no longer GPIO6.3, R16.1
- net PWR_EN: now also R4.2
- net PWR_EN1: now also R8.2
- net PWR_EN2: now also R12.2
- net PWR_EN3: now also R16.2
- net PWR_EN4: now also R20.2
- net PWR_EN5: now also R24.2
Routing:
- net 3.3V1: track 38.8 -> 64.0 mm
- net 3.3V5: track 38.8 -> 64.0 mm
- net 3.3V: track 38.8 -> 64.0 mm
- net 3.3V4: track 38.8 -> 64.0 mm
- net 3.3V2: track 38.8 -> 64.0 mm
- net 3.3V3: track 38.8 -> 64.0 mm
- net PWR_EN5: track 26.8 -> 33.3 mm, vias 1 -> 3
- net PWR_EN4: track 26.8 -> 33.3 mm, vias 1 -> 3
- net PWR_EN3: track 26.8 -> 33.3 mm, vias 1 -> 3
- net PWR_EN1: track 26.8 -> 33.3 mm, vias 1 -> 3
- net PWR_EN: track 26.8 -> 33.3 mm, vias 1 -> 3
- net PWR_EN2: track 26.8 -> 33.3 mm, vias 1 -> 3
- net N$11: track 0.00 -> 5.00 mm
- net N$15: track 0.00 -> 5.00 mm
- net GND5: track 55.8 -> 60.7 mm, vias 95 -> 94
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Other:
- board text added: "x04"
- board text removed: "x03"
